File: V-00735-01.brd (EAGLE design)
At the start: 41 x 73 mm, 32 parts, among them IC2 MAX481CSA, IC3 FT232RL, IC8 ATMEGA644P, Q1 14.7456MHz, X1 MINI-USB-SCHIELD-32005-201

Commit message: v.2.0
Parts:
- added JUM3: S1G3_JUMP, #PaJa_konektory:S1G3_JUM
- added R4, R5: 0R, #PaJa_31:1206
Connections:
- new net +5V_78X: C5.2, IO2.3, JUM3.3, R5.2
- new net +5V_PROG: JUM3.1, R4.2, U$1.2
- net +5V: now also JUM3.2, R4.1, R5.1; no longer C5.2, IO2.3, U$1.4
- net P_MISO: now also U$1.5; no longer U$1.3
- net P_SCK: now also U$1.4; no longer U$1.2
- net RESET: now also U$1.3; no longer U$1.5
Routing:
- net +5V_PROG: track 0.00 -> 24.3 mm
- net +5V_78X: track 0.00 -> 12.6 mm
- net +5V: track 176.7 -> 182.1 mm
- net P_MISO: track 16.3 -> 21.4 mm
- net RESET: track 23.2 -> 18.1 mm, vias 2 -> 0
- net P_SCK: track 15.2 -> 19.9 mm
- net GND: vias 4 -> 8
